File: pcb/right_from_left/keyboard_pcb.kicad_pcb (KiCad board)
At the start: 2 copper layers, 138.8 x 89.9 mm, 48 parts, among them J1 TRRS, J2 Conn_01x04_Male, K0 KEYSW, K1 KEYSW, K10 KEYSW, K11 KEYSW, K12 KEYSW, K13 KEYSW, K14 KEYSW, K15 KEYSW, K2 KEYSW, K20 KEYSW, K21 KEYSW, K22 KEYSW, K23 KEYSW, K24 KEYSW, K25 KEYSW, K3 KEYSW, K30 KEYSW, K31 KEYSW, K32 KEYSW, K4 KEYSW, K5 KEYSW, U1 PCF8574, U2 Pico

Commit message: Revision 1.1 WIP#
Parts:
- removed J2: Conn_01x04_Male, Connector_PinHeader_2.54mm:PinHeader_1x04_P2.54mm_Vertical
- removed MB1, MB2: MountingHole, beekeeb_lib:mousebites_2
- removed MB3, MB4: MountingHole, beekeeb_lib:mousebites_3
- removed R5: 10k, Resistor_SMD:R_0603_1608Metric_Pad0.98x0.95mm_HandSolder
- removed U1: PCF8574, Package_SO:SSOP-20_4.4x6.5mm_P0.65mm
- added C3: 10uF, Capacitor_SMD:C_0603_1608Metric_Pad1.08x0.95mm_HandSolder, F.Cu at (162.0, 108.3)
- added C4: 100nF, Capacitor_SMD:C_0603_1608Metric_Pad1.08x0.95mm_HandSolder, F.Cu at (160.0, 108.3)
- added R10: R, Resistor_SMD:R_0603_1608Metric_Pad0.98x0.95mm_HandSolder, F.Cu at (164.0, 104.7)
- added R11: R, Resistor_SMD:R_0603_1608Metric_Pad0.98x0.95mm_HandSolder, F.Cu at (116.8, 113.2)
- added R12: R, Resistor_SMD:R_0603_1608Metric_Pad0.98x0.95mm_HandSolder, F.Cu at (116.8, 111.5)
- added R13: R, Resistor_SMD:R_0603_1608Metric_Pad0.98x0.95mm_HandSolder, F.Cu at (84.0, 112.8)
- added R14: 10k, Resistor_SMD:R_0603_1608Metric_Pad0.98x0.95mm_HandSolder, F.Cu at (140.5, 114.5)
- added R8: R, Resistor_SMD:R_0603_1608Metric_Pad0.98x0.95mm_HandSolder, F.Cu at (160.0, 104.7)
- added R9: R, Resistor_SMD:R_0603_1608Metric_Pad0.98x0.95mm_HandSolder, F.Cu at (162.0, 104.7)
- added TP1: TestPoint, TestPoint:TestPoint_Pad_D3.0mm, F.Cu at (144.2, 115.2)
- added U3: PCF8574TS, Package_SO:SSOP-20_4.4x6.5mm_P0.65mm, F.Cu at (154.5, 107.5)
- added U4: MCP23009-E/SO, Package_SO:SOIC-18W_7.5x11.6mm_P1.27mm, F.Cu at (143.4, 104.8)
- K0, K1, K10, K11, K12, K13, K14, K15, K2, K20, K21, K22, K23, K24, K25, K3, K30, K31, K32, K4, K5: footprint keyswitches:Kailh_socket_MX_optional_platemount -> keyswitches:Kailh_socket_MX_optional_platemount_3d_pretty_by_datasheet
- R3, R4: footprint Resistor_SMD:R_0603_1608Metric_Pad0.98x0.95mm_HandSolder -> Resistor_SMD:R_0805_2012Metric; moved to B.Cu
- moved R7 25.4 mm to (140.5, 116.2)
- moved C1 16.4 mm to (136.2, 106.0)
- moved C2 16.2 mm to (134.8, 106.0)
- moved R4 11.1 mm to (137.0, 114.0)
- moved R3 10.9 mm to (137.0, 111.8)
- moved R6 8.71 mm to (156.8, 112.8)
- moved D2 3.82 mm to (140.5, 118.2), turned to 0 degrees
- moved D1 3.51 mm to (160.5, 111.8)
- renumbered H1 to H5, H4 to H6, H4 to H7, H4 to H8
Connections:
- C1 pad 1: VCC -> +3.3V
- C2 pad 1: VCC -> +3.3V
- J1 pad 2: VCC -> VBUS
- R3 pad 1: VCC -> +3.3V
- R4 pad 1: VCC -> +3.3V
- U2 pad 1: tx -> rx
- U2 pad 2: rx -> tx
- U2 pad 36: /k04 -> +3.3V
- U2 pad 37: /k05 -> unconnected-(U2-3V3_EN-Pad37)
- U2 pad 39: VCC -> unconnected-(U2-VSYS-Pad39)
- U2 pad 6: unconnected-(U2-GPIO4-Pad6) -> /k05
- U2 pad 7: unconnected-(U2-GPIO5-Pad7) -> /k04
Routing:
- net +3.3V: track 0.00 -> 197.0 mm, vias 0 -> 5
- net VCC: track 141.6 -> 0.00 mm
- net VBUS: track 26.8 -> 86.7 mm
- net /k05: track 23.2 -> 63.0 mm
- net /k04: track 44.2 -> 83.2 mm, vias 0 -> 2
- net Net-(D2-A): track 33.3 -> 2.05 mm, vias 2 -> 0
- net /SDA: track 134.6 -> 158.1 mm
- net /SCL: track 127.2 -> 146.5 mm
- net /LED_A: track 10.7 -> 29.5 mm, vias 0 -> 2
- net /I2C_Int: track 89.4 -> 106.3 mm, vias 1 -> 3
- net /k10: track 72.9 -> 89.0 mm, vias 0 -> 3
- net /LED_B: track 13.0 -> 28.0 mm, vias 0 -> 2
- net /k20: track 61.2 -> 76.0 mm, vias 0 -> 3
- net /k00: track 86.2 -> 99.8 mm
- net /k30: track 43.2 -> 55.8 mm, vias 1 -> 2
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Other:
- outline, holes or cut-outs redrawn
- board text added: "v1.1"
- board text removed: "v1.0"

Commit message: Rev 1.1 WIP
Parts:
- removed C1: 10uF, Capacitor_SMD:C_0603_1608Metric_Pad1.08x0.95mm_HandSolder
- removed C2: 100nF, Capacitor_SMD:C_0603_1608Metric_Pad1.08x0.95mm_HandSolder
- removed U3: PCF8574TS, Package_SO:SSOP-20_4.4x6.5mm_P0.65mm
- C3, C4, R14: moved to B.Cu
- R10, R9: value R -> 10k; moved to B.Cu
- R11, R12, R13, R8: value R -> 10k
- R3, R4: footprint Resistor_SMD:R_0805_2012Metric -> Resistor_SMD:R_0603_1608Metric
- U2: footprint RPi_Pico:RPi_Pico_SMD_TH -> misc:RPi_Pico_SMD_TH
- moved R11 37.8 mm to (124.0, 150.3)
- moved R12 37.8 mm to (124.0, 148.6)
- moved R13 37.8 mm to (91.2, 149.8)
- moved R6 37.8 mm to (164.0, 149.8)
- moved R7 37.8 mm to (147.7, 153.3)
- moved R8 37.8 mm to (167.2, 141.8)
- moved R10 24.0 mm to (140.0, 103.9)
- moved R9 24.0 mm to (138.0, 103.8)
- moved R4 12.2 mm to (143.8, 103.8), turned to 90 degrees
- moved C3 12.0 mm to (150.8, 104.0)
- moved C4 12.0 mm to (148.8, 104.0)
- moved R3 12.0 mm to (146.0, 103.8), turned to 90 degrees
- moved R14 10.7 mm to (141.8, 103.9), turned to 90 degrees
- moved U1 0.67 mm to (143.2, 105.5), turned to -90 degrees
- renumbered U4 to U1
Routing:
- net +3.3V: track 197.0 -> 0.00 mm, vias 5 -> 0
- net /SDA: track 158.1 -> 0.00 mm, vias 2 -> 0
- net /SCL: track 146.5 -> 0.00 mm, vias 2 -> 0
- net /I2C_Int: track 106.3 -> 0.00 mm, vias 3 -> 0
- net /k00: track 99.8 -> 14.6 mm
- net /k32: track 103.0 -> 24.4 mm, vias 2 -> 1
- net /k10: track 89.0 -> 14.4 mm, vias 3 -> 0
- net /k20: track 76.0 -> 14.5 mm, vias 3 -> 0
- net /k31: track 74.0 -> 14.6 mm, vias 2 -> 1
- net /k30: track 55.8 -> 16.2 mm, vias 2 -> 1
- net /LED_A: track 29.5 -> 0.00 mm, vias 2 -> 0
- net /LED_B: track 28.0 -> 0.00 mm, vias 2 -> 0
- net GND: track 73.5 -> 64.1 mm, vias 36 -> 29
- net /MCP_RST: track 9.79 -> 0.71 mm
- net Net-(D1-A): track 2.46 -> 0.23 mm
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